File: Controller/Controller.kicad_sch (KiCad schematic)
At the start: 2 parts, among them U1 COM-09032, U2 COM-09032

Commit message: Fri 24 May 10:03:45 CEST 2024
Parts:
- added SW1: SW_Push, symbol Switch:SW_Push
Other:
- moved on the sheet: U1
Changed lines of the file:
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@@
 	(symbol
 		(lib_id "MyLibs:COM-09032")
-		(at 130.81 83.82 0)
+		(at 140.97 77.47 0)
 		(unit 1)
 		(exclude_from_sim no)
@@
 		(fields_autoplaced yes)
 		(property "Reference" "U1"
-			(at 139.7 87.6299 0)
+			(at 149.86 81.2799 0)
 			(effects
 				(font
@@
 		)
 		(property "Value" "COM-09032"
-			(at 139.7 90.1699 0)
+			(at 149.86 83.8199 0)
 			(effects
 				(font
@@
 		)
 		(property "Footprint" "MyLibs:XDCR_COM-09032"
-			(at 130.81 83.82 0)
+			(at 140.97 77.47 0)
 			(effects
 				(font
@@
 		)
 		(property "Datasheet" ""
-			(at 130.81 83.82 0)
+			(at 140.97 77.47 0)
 			(effects
 				(font
@@
 		)
 		(property "Description" ""
-			(at 130.81 83.82 0)
+			(at 140.97 77.47 0)
 			(effects
 				(font
@@
 		)
 		(property "PARTREV" "N/A"
-			(at 130.81 83.82 0)
+			(at 140.97 77.47 0)
 			(effects
 				(font
@@
 		)
 		(property "STANDARD" "Manufacturer Recommendations"
-			(at 130.81 83.82 0)
+			(at 140.97 77.47 0)
 			(effects
 				(font
@@
 		)
 		(property "MAXIMUM_PACKAGE_HEIGHT" "30.1mm"
-			(at 130.81 83.82 0)
+			(at 140.97 77.47 0)
 			(effects
 				(font
@@
 		)
 		(property "MANUFACTURER" "SparkFun Electronics"
-			(at 130.81 83.82 0)
+			(at 140.97 77.47 0)
 			(effects
 				(font
@@
 					(unit 1)
 				)
+			)
+		)
+	)
+	(symbol
+		(lib_id "Switch:SW_Push")
+		(at 114.3 121.92 0)
+		(unit 1)
+		(exclude_from_sim no)
+		(in_bom yes)
+		(on_board yes)
+		(dnp no)
+		(fields_autoplaced yes)
+		(property "Reference" "SW1"
+			(at 114.3 114.3 0)
+			(effects
+				(font
+					(size 1.27 1.27)
+				)
+			)
+		)
+		(property "Value" "SW_Push"
+			(at 114.3 116.84 0)
+			(effects
+				(font
+					(size 1.27 1.27)
+				)
+			)
+		)
+		(property "Footprint" ""
+			(at 114.3 116.84 0)
+			(effects
+				(font
+					(size 1.27 1.27)
+				)
+				(hide yes)
+			)
+		)
+		(property "Datasheet" "~"
+			(at 114.3 116.84 0)
+			(effects
+				(font
+					(size 1.27 1.27)
+				)
+				(hide yes)
+			)
+		)
+		(property "Description" "Push button switch, generic, two pins"
+			(at 114.3 121.92 0)
+			(effects
+				(font
+					(size 1.27 1.27)
+				)
+				(hide yes)
+			)
+		)
+		(pin "2"
+		)
+		(pin "1"
+		)
+		(instances
+			(project "Controller"
+				(path "/68566f08-c12e-486c-acb3-3400ee298355"
+					(reference "SW1")
+					(unit 1)
+				)
